File: first_pcb.sch (KiCad schematic (older format))
At the start: 64 parts, among them SW1 SW_Push, U1 ATmega32U4-AU, Y1 16MHz

Commit message: Created netlist
Parts:
- C1, C2, C3, C4, C5, C6: footprint (none) -> Capacitor_SMD:C_0805_2012Metric
- C7, D1, D10, D11, D12, D13, D14, D15, D16, D17, D18, D19, D2, D20, D21, D22, D23, D24, D3, D4, D5, D6, D7, D8, D9: footprint (none) -> Diode_SMD:D_SOD-123
- F1: footprint (none) -> MX_Alps_Hybrid:MX-1U
- MX00: renamed from MX1; footprint (none) -> MX_Alps_Hybrid:MX-1U
- MX01: renamed from MX2; footprint (none) -> MX_Alps_Hybrid:MX-1U
- MX02: renamed from MX3; footprint (none) -> MX_Alps_Hybrid:MX-1U
- MX03: renamed from MX4; footprint (none) -> MX_Alps_Hybrid:MX-1U
- MX04: renamed from MX5; footprint (none) -> MX_Alps_Hybrid:MX-1U
- MX05: renamed from MX6; footprint (none) -> MX_Alps_Hybrid:MX-1U
- MX10: renamed from MX7; footprint (none) -> MX_Alps_Hybrid:MX-1U
- MX11: renamed from MX8; footprint (none) -> MX_Alps_Hybrid:MX-1U
- MX12: renamed from MX9; footprint (none) -> MX_Alps_Hybrid:MX-1U
- MX13: renamed from MX10; footprint (none) -> MX_Alps_Hybrid:MX-1U
- MX14: renamed from MX11; footprint (none) -> MX_Alps_Hybrid:MX-1U
- MX15: renamed from MX12; footprint (none) -> MX_Alps_Hybrid:MX-1U
- MX20: renamed from MX13; footprint (none) -> MX_Alps_Hybrid:MX-1U
- MX21: renamed from MX14; footprint (none) -> MX_Alps_Hybrid:MX-1U
- MX22: renamed from MX15; footprint (none) -> MX_Alps_Hybrid:MX-1U
- MX23: renamed from MX16; footprint (none) -> MX_Alps_Hybrid:MX-1U
- MX24: renamed from MX17; footprint (none) -> MX_Alps_Hybrid:MX-1U
- MX25: renamed from MX18; footprint (none) -> MX_Alps_Hybrid:MX-1U
- MX30: renamed from MX19; footprint (none) -> MX_Alps_Hybrid:MX-1U
- MX31: renamed from MX20; footprint (none) -> MX_Alps_Hybrid:MX-1U
- MX32: renamed from MX21; footprint (none) -> MX_Alps_Hybrid:MX-1U
- MX33: renamed from MX22; footprint (none) -> MX_Alps_Hybrid:MX-1U
- MX34: renamed from MX23; footprint (none) -> MX_Alps_Hybrid:MX-1U
- MX35: renamed from MX24; footprint (none) -> MX_Alps_Hybrid:MX-1U
- R1, R2, R3, R4: footprint (none) -> Resistor_SMD:R_0805_2012Metric_Pad1.15x1.40mm_HandSolder
- SW1: footprint (none) -> random-keyboard-parts:SKQG-1155865
- USB1: footprint (none) -> random-keyboard-parts:Molex-0548190589
- Y1: footprint (none) -> Crystal:Crystal_SMD_3225-4Pin_3.2x2.5mm_HandSoldering

Commit message: Updated pcb
Parts:
- F1: footprint MX_Alps_Hybrid:MX-1U -> Fuse:Fuse_1206_3216Metric_Pad1.42x1.75mm_HandSolder
Changed lines of the file:
@@
 F 0 "F1" V 5145 1225 50  0000 C CNN
 F 1 "500mA" V 5236 1225 50  0000 C CNN
-F 2 "MX_Alps_Hybrid:MX-1U" H 5400 1025 50  0001 L CNN
+F 2 "Fuse:Fuse_1206_3216Metric_Pad1.42x1.75mm_HandSolder" H 5400 1025 50  0001 L CNN
 F 3 "~" H 5350 1225 50  0001 C CNN
 	1    5350 1225
